Commit message: test the boxsides ob

File: src/yumi/yumi_description/urdf/workspace.xacro (robot description, xacro)
@@ -19,5 +19,5 @@
       <visual>
         <geometry>
-          <box size="1.6 0.8 0.026"/>
+          <box size="0.1 0.8 0.026"/>
         </geometry>
         <origin rpy="0 0 0" xyz="0 0 0"/>
@@ -26,5 +26,5 @@
       <collision>
         <geometry>
-          <box size="1.6 0.8 0.026"/>
+          <box size="0.1 0.8 0.026"/>
         </geometry>
         <origin rpy="0 0 0" xyz="0 0 0"/>

Commit message: modified the workspace URDF model using sketchup

File: src/yumi/yumi_description/urdf/workspace.xacro (robot description, xacro)
@@ -19,38 +19,38 @@
       <visual>
         <geometry>
-          <box size="0.1 0.8 0.026"/>
+          <box size="1.2 0.8 0.026"/>
         </geometry>
-        <origin rpy="0 0 0" xyz="0 0 0"/>
+        <origin rpy="0 0 0" xyz="0 0 -0.115"/>
         <material name="Ivory"/>
       </visual>
       <collision>
         <geometry>
-          <box size="0.1 0.8 0.026"/>
+          <box size="1.2 0.8 0.026"/>
         </geometry>
-        <origin rpy="0 0 0" xyz="0 0 0"/>
+        <origin rpy="0 0 0" xyz="0 0 -0.115"/>
         <material name="Ivory"/>
       </collision>
     </link>
-    <!--<joint name="table_two_to_${table_parent}" type="fixed">
+    <joint name="box_to_${table_parent}" type="fixed">
       <parent link="${table_parent}"/>
-      <child link="table_two"/>
-      <origin rpy="0 0 0" xyz="-0.4 1.3 0"/>
-    </joint>-->
-    <!--<link name="table_two">
+      <child link="box"/>
+      <origin rpy="0 0 0" xyz="0 0 0"/>
+    </joint>
+    <link name="box">
       <visual>
+        <origin rpy="0 0 0" xyz="0.25 -0.15 -0.115"/>
         <geometry>
-          <box size="0.8 1.8 0.026"/>
+          <mesh filename="package://yumi_description/meshes/workspace/box_su.stl"/>
         </geometry>
-        <origin rpy="0 0 0" xyz="0 0 0"/>
-        <material name="Ivory"/>
+        <material name="Blue"/>
       </visual>
       <collision>
+        <origin rpy="0 0 0" xyz="0.25 -0.15 -0.115"/>
         <geometry>
-          <box size="0.8 1.8 0.026"/>
+          <mesh filename="package://yumi_description/meshes/workspace/box_su.stl"/>
         </geometry>
-        <origin rpy="0 0 0" xyz="0 0 0"/>
-        <material name="Ivory"/>
+        <material name="Blue"/>
       </collision>
-    </link>-->
+    </link>
     <!--                         -->
     <!--       YUMI STAND        -->
@@ -63,15 +63,15 @@
     <link name="stand">
       <visual>
-        <origin rpy="0 0 0" xyz="165.03939 -0.25716 0.00014"/>
-        <origin rpy="0 0 0" xyz=""/>
+        <origin rpy="0 0 ${PI}" xyz="0.13 0 -0.1525"/>
+        <origin rpy="0 0 ${PI}" xyz=""/>
         <geometry>
-          <mesh filename="package://yumi_description/meshes/base/IRB14000_BaseStand_Fixed.stl"/>
+          <mesh filename="package://yumi_description/meshes/base/IRB14000_BaseStand_Fixed_own.stl"/>
         </geometry>
         <material name="Ivory"/>
       </visual>
       <collision>
-        <origin rpy="0 0 0" xyz="165.03939 -0.25716 0.00014"/>
+        <origin rpy="0 0 ${PI}" xyz="0.13 0 -0.1525"/>
         <geometry>
-          <mesh filename="package://yumi_description/meshes/base/IRB14000_BaseStand_Fixed.stl"/>
+          <mesh filename="package://yumi_description/meshes/base/IRB14000_BaseStand_Fixed_own.stl"/>
         </geometry>
         <material name="Ivory"/>

Commit message: modified the obj of planning scence and first test of picking postcard

File: src/yumi/yumi_description/urdf/workspace.xacro (robot description, xacro)
@@ -1,7 +1,7 @@
 <?xml version="1.0"?>
 <!--
-  PROGRAMMER: Frederick Wachter
-  DATE CREATED: 2016-05-30
-  LAST MODIFIED: 2016-05-30
+  PROGRAMMER: Honghao Lv
+  DATE CREATED: 2019-04-20
+  LAST MODIFIED: 2019-04-21
   PURPOSE: Build the workspace around YuMi
 -->
@@ -37,5 +37,5 @@
       <origin rpy="0 0 0" xyz="0 0 0"/>
     </joint>
-    <link name="box">
+    <!--<link name="box">
       <visual>
         <origin rpy="0 0 0" xyz="0.25 -0.15 -0.115"/>
@@ -43,5 +43,5 @@
           <mesh filename="package://yumi_description/meshes/workspace/box_su.stl"/>
         </geometry>
-        <material name="Blue"/>
+        <material name="Ivory"/>
       </visual>
       <collision>
@@ -50,5 +50,21 @@
           <mesh filename="package://yumi_description/meshes/workspace/box_su.stl"/>
         </geometry>
-        <material name="Blue"/>
+        <material name="Ivory"/>
+      </collision>
+    </link>-->
+        <link name="box">
+      <visual>
+        <origin rpy="0 0 0" xyz="0.4 0 -0.09"/>
+        <geometry>
+          <box size="0.5 0.5 0.05"/>
+        </geometry>
+        <material name="Ivory"/>
+      </visual>
+      <collision>
+        <origin rpy="0 0 0" xyz="0.4 0 -0.09"/>
+        <geometry>
+          <box size="0.5 0.5 0.05"/>
+        </geometry>
+        <material name="Ivory"/>
       </collision>
     </link>
@@ -63,5 +79,5 @@
     <link name="stand">
       <visual>
-        <origin rpy="0 0 ${PI}" xyz="0.13 0 -0.1525"/>
+        <origin rpy="0 0 ${PI}" xyz="0.14 0 -0.1525"/>
         <origin rpy="0 0 ${PI}" xyz=""/>
         <geometry>
@@ -71,5 +87,5 @@
       </visual>
       <collision>
-        <origin rpy="0 0 ${PI}" xyz="0.13 0 -0.1525"/>
+        <origin rpy="0 0 ${PI}" xyz="0.14 0 -0.1525"/>
         <geometry>
           <mesh filename="package://yumi_description/meshes/base/IRB14000_BaseStand_Fixed_own.stl"/>

Commit message: finish a test of an programming process of yumi control of 10 position for left/right arms

File: src/yumi/yumi_description/urdf/workspace.xacro (robot description, xacro)
@@ -21,5 +21,5 @@
           <box size="1.2 0.8 0.026"/>
         </geometry>
-        <origin rpy="0 0 0" xyz="0 0 -0.115"/>
+        <origin rpy="0 0 0" xyz="0.05 0 -0.115"/>
         <material name="Ivory"/>
       </visual>
@@ -28,5 +28,5 @@
           <box size="1.2 0.8 0.026"/>
         </geometry>
-        <origin rpy="0 0 0" xyz="0 0 -0.115"/>
+        <origin rpy="0 0 0" xyz="0.05 0 -0.115"/>
         <material name="Ivory"/>
       </collision>
@@ -55,14 +55,14 @@
         <link name="box">
       <visual>
-        <origin rpy="0 0 0" xyz="0.4 0 -0.09"/>
+        <origin rpy="0 0 0" xyz="0.55 0 -0.085"/>
         <geometry>
-          <box size="0.5 0.5 0.05"/>
+          <box size="0.2 0.55 0.04"/>
         </geometry>
         <material name="Ivory"/>
       </visual>
       <collision>
-        <origin rpy="0 0 0" xyz="0.4 0 -0.09"/>
+        <origin rpy="0 0 0" xyz="0.55 0 -0.085"/>
         <geometry>
-          <box size="0.5 0.5 0.05"/>
+          <box size="0.2 0.55 0.04"/>
         </geometry>
         <material name="Ivory"/>

File: src/yumi/yumi_description/urdf/yumi_servo_gripper.xacro (robot description, xacro)
@@ -53,5 +53,5 @@
       <origin xyz="0 -0.0065 0.0837" rpy="${-PI/2} 0 0"/>
       <axis xyz="-1 0 0"/>
-      <limit lower="0" upper="0.024" effort="${max_effort}" velocity="0.02" />
+      <limit lower="0" upper="0.0245" effort="${max_effort}" velocity="0.02" />
       <dynamics damping="${joint_damping}"/>
     </joint>
@@ -82,5 +82,5 @@
       <origin xyz="0 0.0065 0.0837" rpy="0 0 ${PI}"/>
       <axis xyz="-1 0 0"/>
-      <limit lower="0" upper="0.024" effort="${max_effort}" velocity="0.02" />
+      <limit lower="0" upper="0.0245" effort="${max_effort}" velocity="0.02" />
       <dynamics damping="${joint_damping}"/>
       <mimic joint="${name}_joint_r"/>

File: src/yumi/yumi_description/urdf/yumi_servo_gripper_left.xacro (robot description, xacro)
@@ -53,5 +53,5 @@
       <origin xyz="0 -0.0065 0.0837" rpy="${PI/2} 0 0"/>
       <axis xyz="-1 0 0"/>
-      <limit lower="0" upper="0.024" effort="${max_effort}" velocity="0.02" />
+      <limit lower="0" upper="0.025" effort="${max_effort}" velocity="0.02" />
       <dynamics damping="${joint_damping}"/>
     </joint>
@@ -82,5 +82,5 @@
       <origin xyz="0 0.0065 0.0837" rpy="0 0 ${PI}"/>
       <axis xyz="-1 0 0"/>
-      <limit lower="0" upper="0.024" effort="${max_effort}" velocity="0.02" />
+      <limit lower="0" upper="0.025" effort="${max_effort}" velocity="0.02" />
       <dynamics damping="${joint_damping}"/>
       <mimic joint="${name}_joint_r"/>
