Commit message: 20190719commitbefore indin

File: src/yumi/yumi_description/urdf/yumi_servo_gripper.xacro (robot description, xacro)
@@ -53,5 +53,5 @@
       <origin xyz="0 -0.0065 0.0837" rpy="${-PI/2} 0 0"/>
       <axis xyz="-1 0 0"/>
-      <limit lower="0" upper="0.0245" effort="${max_effort}" velocity="0.02" />
+      <limit lower="0" upper="0.025" effort="${max_effort}" velocity="0.02" />
       <dynamics damping="${joint_damping}"/>
     </joint>
@@ -82,5 +82,5 @@
       <origin xyz="0 0.0065 0.0837" rpy="0 0 ${PI}"/>
       <axis xyz="-1 0 0"/>
-      <limit lower="0" upper="0.0245" effort="${max_effort}" velocity="0.02" />
+      <limit lower="0" upper="0" effort="${max_effort}" velocity="0.02" />
       <dynamics damping="${joint_damping}"/>
       <mimic joint="${name}_joint_r"/>

Commit message: the first demo test for ZhangZhiyu

File: src/yumi/yumi_description/urdf/yumi_servo_gripper.xacro (robot description, xacro)
@@ -82,5 +82,5 @@
       <origin xyz="0 0.0065 0.0837" rpy="0 0 ${PI}"/>
       <axis xyz="-1 0 0"/>
-      <limit lower="0" upper="0" effort="${max_effort}" velocity="0.02" />
+      <limit lower="0" upper="0.025" effort="${max_effort}" velocity="0.02" />
       <dynamics damping="${joint_damping}"/>
       <mimic joint="${name}_joint_r"/>
